Commit message: modified doosan robot color

File: pykin/asset/urdf/doosan/doosan.urdf (robot description, URDF)
Before this commit: robot a0509, 7 links, 6 joints
Links:
- added link doosan_controller_box; collision box size=0.22 0.4 0.53
- added link doosan_pedestal, mass 60.86397744; collision cylinder length=0.62 radius=0.18; visual mesh filename=meshes/doosan_pedestal/pedestal.STL
- added link doosan_pedestal_feet; collision box size=0.77 0.7 0.31
Joints:
- added joint doosan_controller_box_fixed: type fixed, parent base_0, child doosan_controller_box, origin xyz=0.0 0.0 0.0 rpy=0 0 0
- added joint doosan_pedestal_feet_fixed: type fixed, parent base_0, child doosan_pedestal_feet, origin xyz=0.0 0.0 0.0 rpy=0 0 0
- added joint doosan_pedestal_fixed: type fixed, parent base_0, child doosan_pedestal, origin xyz=0.0 0.0 0.0 rpy=0 0 0

Commit message: added doosan robot

File: pykin/asset/urdf/doosan/doosan.urdf (robot description, URDF)
Before this commit: robot a0509, 10 links, 9 joints
Links:
- link base_0: mass 2.198 -> 3.635; geometry visual mesh filename=meshes/a0912_blue/A0912_0_0.stl scale=0.001 0.001 0.001
- link link1: mass 3.715 -> 7.863; geometry collision cylinder length=0.2 radius=0.08; visual mesh filename=meshes/a0912_blue/A0912_1_0.stl scale=0.001 0.001 0.001
- link link2: mass 6.837 -> 10.985; geometry collision cylinder length=0.6 radius=0.08; visual mesh filename=meshes/a0912_blue/A0912_2_0.stl scale=0.001 0.001 0.001
- link link3: mass 2.769 -> 2.881; geometry visual mesh filename=meshes/a0912_blue/A0912_3_0.stl scale=0.001 0.001 0.001; visual mesh filename=meshes/a0912_blue/A0912_3_1.stl scale=0.001 0.001 0.001
- link link4: mass 2.679 -> 3.273; geometry collision cylinder length=0.4 radius=0.05; visual mesh filename=meshes/a0912_blue/A0912_4_0.stl scale=0.001 0.001 0.001
- link link5: mass 2.051 -> 2.141; geometry collision cylinder length=0.15 radius=0.06; visual mesh filename=meshes/a0912_blue/A0912_5_0.stl scale=0.001 0.001 0.001
- link link6: mass 0.773 -> 0.784; geometry visual mesh filename=meshes/a0912_blue/A0912_6_0.stl scale=0.001 0.001 0.001
Joints:
- joint joint1: limit lower=-6.2832 upper=6.2832 effort=194 velocity=3.1416 -> lower=-6.2832 upper=6.2832 effort=411 velocity=3.1416; origin xyz=0 0 0.1555 rpy=0 0 0 -> xyz=0 0 0.195 rpy=0 0 0
- joint joint2: limit lower=-6.2832 upper=6.2832 effort=194 velocity=3.1416 -> lower=-6.2832 upper=6.2832 effort=411 velocity=3.1416; origin xyz=0 0 0 rpy=0 -1.571 -1.571 -> xyz=0 0.039 0 rpy=0 -1.571 -1.571
- joint joint3: limit lower=-2.7925 upper=2.7925 effort=163 velocity=3.1416 -> lower=-2.7925 upper=2.7925 effort=194 velocity=3.1416; origin xyz=0.409 0 0 rpy=0 0 1.571 -> xyz=0.56 0 0 rpy=0 0 1.571
- joint joint4: origin xyz=0 -0.367 0 rpy=1.571 0 0 -> xyz=0 -0.516 0 rpy=1.571 0 0
