Commit message: added robotiq 140 gripper

File: pykin/asset/urdf/doosan/doosan_with_robotiq140.urdf (robot description, URDF)
Before this commit: robot iiwa7, 23 links, 22 joints
Links:
- removed link iiwa7_controller_box
- removed link iiwa7_link_0
- removed link iiwa7_link_1
- removed link iiwa7_link_2
- removed link iiwa7_link_3
- removed link iiwa7_link_4
- removed link iiwa7_link_5
- removed link iiwa7_link_6
- removed link iiwa7_link_7
- removed link iiwa7_pedestal
- removed link iiwa7_pedestal_feet
- removed link iiwa7_right_hand
- added link base_0, mass 3.635; visual mesh filename=meshes/a0912_blue/A0912_0_0.stl scale=0.001 0.001 0.001
- added link doosan_controller_box; collision box size=0.22 0.4 0.53
- added link doosan_pedestal, mass 60.86397744; collision cylinder length=0.62 radius=0.18; visual mesh filename=meshes/doosan_pedestal/pedestal.STL
- added link doosan_pedestal_feet; collision box size=0.77 0.7 0.31
- added link doosan_right_hand
- added link link1, mass 7.863; collision cylinder length=0.2 radius=0.08; visual mesh filename=meshes/a0912_blue/A0912_1_0.stl scale=0.001 0.001 0.001
- added link link2, mass 10.985; collision cylinder length=0.6 radius=0.08; visual mesh filename=meshes/a0912_blue/A0912_2_0.stl scale=0.001 0.001 0.001
- added link link3, mass 2.881; visual mesh filename=meshes/a0912_blue/A0912_3_0.stl scale=0.001 0.001 0.001; visual mesh filename=meshes/a0912_blue/A0912_3_1.stl scale=0.001 0.001 0.001
- added link link4, mass 3.273; collision cylinder length=0.4 radius=0.05; visual mesh filename=meshes/a0912_blue/A0912_4_0.stl scale=0.001 0.001 0.001
- added link link5, mass 2.141; collision cylinder length=0.15 radius=0.06; visual mesh filename=meshes/a0912_blue/A0912_5_0.stl scale=0.001 0.001 0.001
- added link link6, mass 0.784; visual mesh filename=meshes/a0912_blue/A0912_6_0.stl scale=0.001 0.001 0.001
Joints:
- removed joint iiwa7_controller_box_fixed
- removed joint iiwa7_joint_1
- removed joint iiwa7_joint_2
- removed joint iiwa7_joint_3
- removed joint iiwa7_joint_4
- removed joint iiwa7_joint_5
- removed joint iiwa7_joint_6
- removed joint iiwa7_joint_7
- removed joint iiwa7_pedestal_feet_fixed
- removed joint iiwa7_pedestal_fixed
- removed joint iiwa7_right_gripper_fixed
- removed joint iiwa7_right_hand_fixed
- added joint doosan_controller_box_fixed: type fixed, parent base_0, child doosan_controller_box, origin xyz=0.0 0.0 0.0 rpy=0 0 0
- added joint doosan_pedestal_feet_fixed: type fixed, parent base_0, child doosan_pedestal_feet, origin xyz=0.0 0.0 0.0 rpy=0 0 0
- added joint doosan_pedestal_fixed: type fixed, parent base_0, child doosan_pedestal, origin xyz=0.0 0.0 0.0 rpy=0 0 0
- added joint doosan_right_gripper_fixed: type fixed, parent doosan_right_hand, child right_gripper, origin xyz=0 0 -0.0625, axis 0 0 0
- added joint doosan_right_hand_fixed: type fixed, parent link6, child doosan_right_hand, origin xyz=0 0 0 rpy=0 0 0
- added joint joint1: type revolute, parent base_0, child link1, origin xyz=0 0 0.195 rpy=0 0 0, axis 0 0 1, limit lower=-6.2832 upper=6.2832 effort=411 velocity=3.1416
- added joint joint2: type revolute, parent link1, child link2, origin xyz=0 0.039 0 rpy=0 -1.571 -1.571, axis 0 0 1, limit lower=-6.2832 upper=6.2832 effort=411 velocity=3.1416
- added joint joint3: type revolute, parent link2, child link3, origin xyz=0.56 0 0 rpy=0 0 1.571, axis 0 0 1, limit lower=-2.7925 upper=2.7925 effort=194 velocity=3.1416
- added joint joint4: type revolute, parent link3, child link4, origin xyz=0 -0.516 0 rpy=1.571 0 0, axis 0 0 1, limit lower=-6.2832 upper=6.2832 effort=50 velocity=6.2832
- added joint joint5: type revolute, parent link4, child link5, origin xyz=0 0 0 rpy=-1.571 0 0, axis 0 0 1, limit lower=-6.2832 upper=6.2832 effort=50 velocity=6.2832
- added joint joint6: type revolute, parent link5, child link6, origin xyz=0 -0.124 0 rpy=1.571 0 0, axis 0 0 1, limit lower=-6.2832 upper=6.2832 effort=50 velocity=6.2832

File: pykin/asset/urdf/gripper/robotiq_140_gripper.urdf (robot description, URDF)
Before this commit: robot iiwa7, 23 links, 22 joints
Links:
- removed link iiwa7_controller_box
- removed link iiwa7_link_0
- removed link iiwa7_link_1
- removed link iiwa7_link_2
- removed link iiwa7_link_3
- removed link iiwa7_link_4
- removed link iiwa7_link_5
- removed link iiwa7_link_6
- removed link iiwa7_link_7
- removed link iiwa7_pedestal
- removed link iiwa7_pedestal_feet
- removed link iiwa7_right_hand
Joints:
- removed joint iiwa7_controller_box_fixed
- removed joint iiwa7_joint_1
- removed joint iiwa7_joint_2
- removed joint iiwa7_joint_3
- removed joint iiwa7_joint_4
- removed joint iiwa7_joint_5
- removed joint iiwa7_joint_6
- removed joint iiwa7_joint_7
- removed joint iiwa7_pedestal_feet_fixed
- removed joint iiwa7_pedestal_fixed
- removed joint iiwa7_right_gripper_fixed
- removed joint iiwa7_right_hand_fixed
- added joint doosan_right_gripper_fixed: type fixed, parent doosan_right_hand, child right_gripper, origin xyz=0 0 -0.0625, axis 0 0 0

File: pykin/asset/urdf/panda/panda.urdf (robot description, URDF)
Before this commit: robot panda, 16 links, 15 joints
Joints:
- removed joint panda_right_right_gripper_fixed
- added joint panda_right_gripper_fixed: type fixed, parent panda_right_hand, child right_gripper, origin xyz=0 0 0 rpy=0 0 -1.5707963, axis 0 0 0

Commit message: added robot_fk_doosan_test.py

File: pykin/asset/urdf/doosan/doosan_with_robotiq140.urdf (robot description, URDF)
Before this commit: robot doosan, 22 links, 21 joints
Links:
- removed link doosan_right_hand
- added link right_hand
- added link tcp
Joints:
- removed joint doosan_right_gripper_fixed
- removed joint doosan_right_hand_fixed
- added joint doosan_eef_fixed: type fixed, parent right_gripper, child tcp, origin xyz=0 0 -0.27
- added joint right_gripper_fixed: type fixed, parent right_hand, child right_gripper, origin xyz=0 0 -0.0625, axis 0 0 0
- added joint right_hand_fixed: type fixed, parent link6, child right_hand, origin xyz=0 0 0 rpy=0 0 0

File: pykin/asset/urdf/panda/panda.urdf (robot description, URDF)
Before this commit: robot panda, 16 links, 15 joints
Links:
- removed link panda_right_hand
- added link right_hand
Joints:
- removed joint panda_right_hand_fixed
- added joint right_hand_fixed: type fixed, parent panda_link_7, child right_hand, origin xyz=0 0 0.1065 rpy=0 0 -0.7858908
- joint panda_eef_fixed: parent panda_right_hand -> right_hand
- joint panda_right_gripper_fixed: parent panda_right_hand -> right_hand

Commit message: modified gripper.py

File: pykin/asset/urdf/doosan/doosan_with_robotiq140.urdf (robot description, URDF)
Before this commit: robot doosan, 23 links, 22 joints
Joints:
- joint doosan_eef_fixed: origin xyz=0 0 -0.27 -> xyz=0 0 0.2075; parent right_gripper -> right_hand
- joint right_hand_fixed: origin xyz=0 0 0 rpy=0 0 0 -> xyz=0 0 0 rpy=0 0 -1.5707963

Commit message: modified doosan gripper

File: pykin/asset/urdf/doosan/doosan_with_robotiq140.urdf (robot description, URDF)
Before this commit: robot doosan, 23 links, 22 joints
Links:
- added link collision_pad; collision box size=0.02 0.012 0.275
- link left_inner_finger_pad: geometry collision box size=0.03 0.07 0.0375; visual box size=0.027 0.065 0.0075
- link right_inner_finger_pad: geometry collision box size=0.03 0.07 0.0375; visual box size=0.027 0.065 0.0075
Joints:
- added joint collision_pad_joint: type fixed, parent left_inner_finger, child collision_pad, origin xyz=0 -0.0057554 -0.12203 rpy=0 0 0, axis 0 0 1
