Commit message: modified fanuc

File: pykin/assets/urdf/fanuc/fanuc_r2000ic_165f.urdf (robot description, URDF)
Before this commit: robot fanuc_r2000ic_165f, 10 links, 9 joints
Links:
- removed link base
- removed link flange
- removed link tool0
Joints:
- removed joint base_link-base
- removed joint joint_6-flange
- removed joint link_6-tool0

Commit message: modified fanuc urdf

File: pykin/assets/urdf/fanuc/fanuc_r2000ic_165f.urdf (robot description, URDF)
Before this commit: robot fanuc_r2000ic_165f, 7 links, 6 joints
Joints:
- joint joint_4: axis -1 0 0 -> 1 0 0
- joint joint_6: axis -1 0 0 -> 0 0 1; origin xyz=0.215 0 0 rpy=0 0 0 -> xyz=0.215 0 0 rpy=0 1.5707963267948966192313216916398 0
